Commit message: world

File: description/lidar.xacro (robot description, xacro)
@@ -6,4 +6,49 @@
         <origin xyz="0.1 0 0.175" rpy="0 0 0"/>
     </joint>
-    <link></link>
+    <link name="laser_frame">
+         <visual>
+            <geometry>
+                <box size="0.05 0.05 0.070"/>
+            </geometry>
+            <material name="red"/>
+        </visual>
+        <collision>
+            <geometry>
+                <box size="0.05 0.05 0.070"/>
+            </geometry>
+        </collision>
+        <xacro:inertial_box mass="0.16" x="0.05" y="0.05" z="0.070">
+            <origin xyz="0 0 0" rpy="0 0 0"/>
+        </xacro:inertial_box>
+    </link>
+    <gazebo reference="laser_frame">
+        <material>Gazebo/Red</material>
+        <sensor name="laser" type="ray">
+            <pose> 0 0 0 0 0 0 </pose>
+            <visualize>true</visualize>
+            <update_rate>10</update_rate>
+            <ray>
+                <scan>
+                    <horizontal>
+                        <samples>360</samples>
+                        <resolution>0.36</resolution>
+                        <min_angle>-50</min_angle>
+                        <max_angle>50</max_angle>
+                    </horizontal>
+                    <range>
+                        <min>0.02</min>
+                        <max>4</max>
+                        <resolution>0.01</resolution>
+                    </range>
+                </scan>
+            </ray>
+            <plugin name="laser_controller" filename="libgazebo_ros_ray_sensor.so">
+                <ros>
+                    <argument>~/out:=scan</argument>
+                </ros>
+                <output_type>sensor_msgs/LaserScan</output_type>
+                <frame_name>laser_frame</frame_name>
+            </plugin>
+        </sensor>
+    </gazebo>
 </robot>

File: description/robot_core.xacro (robot description, xacro)
@@ -11,4 +11,7 @@
         <color rgba="0.2 0.2 1 1" />
     </material>
+    <material name="red">
+        <color rgba="1 0 0 1" />
+    </material>
     <material name="black">
         <color rgba="0 0 0 1" />
@@ -21,11 +24,11 @@
         <parent link="base_link"/>
         <child link="chassis"/>
-        <origin xyz="-0.1 0 0"/>
+        <origin xyz="1 1 0"/>
     </joint>
     <link name="chassis">
         <visual>
-            <origin xyz="0.15 0 0.075"/>
+            <origin xyz="0 0 0.007"/>
             <geometry>
-                <box size="0.3 0.3 0.15"/>
+                <box size="0.140 0.1778 0.0455"/>
             </geometry>
             <material name="white"/>
@@ -34,8 +37,8 @@
             <origin xyz="0.15 0 0.075"/>
             <geometry>
-                <box size="0.3 0.3 0.15"/>
+                <box size="0.140 0.1778 0.0455"/>
             </geometry>
         </collision>
-        <xacro:inertial_box mass="0.5" x="0.3" y="0.3" z="0.15">
+        <xacro:inertial_box mass="0.5" x="0.140" y="0.1778" z="0.0455">
             <origin xyz="0.15 0 0.075" rpy="0 0 0"/>
         </xacro:inertial_box>
@@ -46,7 +49,7 @@
     <!--  LEFT WHEEL LINK  -->
     <joint name="left_wheel_joint" type="continuous">
-        <parent link="base_link"/>
+        <parent link="chassis"/>
         <child link="left_wheel"/>
-        <origin xyz="0 0.175 0" rpy="-${pi/2} 0 0"/>
+        <origin xyz="0 0.1016 0" rpy="-${pi/2} 0 0"/>
         <axis xyz="0 0 1"/>
     </joint>
@@ -54,5 +57,5 @@
         <visual>
             <geometry>
-                <cylinder radius="0.05" length="0.04"/>
+                <cylinder radius="0.034" length="0.0254"/>
             </geometry>
             <material name="blue"/>
@@ -60,9 +63,9 @@
         <collision>
             <geometry>
-                <cylinder radius="0.05" length="0.04"/>
+                <cylinder radius="0.034" length="0.0254"/>
             </geometry>
         </collision>
-        <xacro:inertial_cylinder mass="0.1" length="0.04" radius="0.05">
-            <origin xyz="0 0 0" rpy="0 0 0"/>
+        <xacro:inertial_cylinder mass="0.1" length="0.0254" radius="0.034">
+            <origin xyz="0 0 0.027" rpy="0 0 0"/>
         </xacro:inertial_cylinder>
     </link>
@@ -72,7 +75,7 @@
     <!--  RIGHT WHEEL LINK  -->
     <joint name="right_wheel_joint" type="continuous">
-        <parent link="base_link"/>
+        <parent link="chassis"/>
         <child link="right_wheel"/>
-        <origin xyz="0 -0.175 0" rpy="${pi/2} 0 0"/>
+        <origin xyz="0 -0.1016 0" rpy="${pi/2} 0 0"/>
         <axis xyz="0 0 -1"/>
     </joint>
@@ -80,5 +83,5 @@
         <visual>
             <geometry>
-                <cylinder radius="0.05" length="0.04"/>
+                <cylinder radius="0.034" length="0.0254"/>
             </geometry>
             <material name="blue"/>
@@ -86,9 +89,9 @@
         <collision>
             <geometry>
-                <cylinder radius="0.05" length="0.04"/>
+                <cylinder radius="0.034" length="0.0254"/>
             </geometry>
         </collision>
-        <xacro:inertial_cylinder mass="0.1" length="0.04" radius="0.05">
-            <origin xyz="0 0 0" rpy="0 0 0"/>
+        <xacro:inertial_cylinder mass="0.1" length="0.0254" radius="0.034">
+            <origin xyz="0 0 0.027" rpy="0 0 0"/>
         </xacro:inertial_cylinder>
     </link>

Commit message: simulation géométrie roue +corp +lidar ok

File: description/lidar.xacro (robot description, xacro)
@@ -4,5 +4,5 @@
         <parent link="chassis"/>
         <child link="laser_frame"/>
-        <origin xyz="0.1 0 0.175" rpy="0 0 0"/>
+        <origin xyz="0.03 0 0.065" rpy="-${pi} 0 0"/>
     </joint>
     <link name="laser_frame">
@@ -31,15 +31,15 @@
                 <scan>
                     <horizontal>
-                        <samples>360</samples>
+                        <samples>240</samples>
                         <resolution>0.36</resolution>
-                        <min_angle>-50</min_angle>
-                        <max_angle>50</max_angle>
+                        <min_angle>-3.14</min_angle>
+                        <max_angle>3.14</max_angle>
                     </horizontal>
-                    <range>
-                        <min>0.02</min>
-                        <max>4</max>
-                        <resolution>0.01</resolution>
-                    </range>
                 </scan>
+                <range>
+                    <min>0.04</min>
+                    <max>4</max>
+                    <resolution>1</resolution>
+                </range>
             </ray>
             <plugin name="laser_controller" filename="libgazebo_ros_ray_sensor.so">

File: description/robot_core.xacro (robot description, xacro)
@@ -24,5 +24,5 @@
         <parent link="base_link"/>
         <child link="chassis"/>
-        <origin xyz="1 1 0"/>
+        <origin xyz="0 0 0"/>
     </joint>
     <link name="chassis">
@@ -30,16 +30,16 @@
             <origin xyz="0 0 0.007"/>
             <geometry>
-                <box size="0.140 0.1778 0.0455"/>
+                <box size="0.140 0.320 0.0455"/>
             </geometry>
             <material name="white"/>
         </visual>
         <collision>
-            <origin xyz="0.15 0 0.075"/>
+            <origin xyz="0 0 0.007"/>
             <geometry>
-                <box size="0.140 0.1778 0.0455"/>
+                <box size="0.140 0.320 0.0455"/>
             </geometry>
         </collision>
-        <xacro:inertial_box mass="0.5" x="0.140" y="0.1778" z="0.0455">
-            <origin xyz="0.15 0 0.075" rpy="0 0 0"/>
+        <xacro:inertial_box mass="0.5" x="0.140" y="0.320" z="0.0455">
+            <origin xyz="0.004 0.001 0.051" rpy="0 0 0"/>
         </xacro:inertial_box>
     </link>
@@ -51,5 +51,5 @@
         <parent link="chassis"/>
         <child link="left_wheel"/>
-        <origin xyz="0 0.1016 0" rpy="-${pi/2} 0 0"/>
+        <origin xyz="0 0.1016 0.00425" rpy="-${pi/2} 0 0"/>
         <axis xyz="0 0 1"/>
     </joint>
@@ -67,5 +67,5 @@
         </collision>
         <xacro:inertial_cylinder mass="0.1" length="0.0254" radius="0.034">
-            <origin xyz="0 0 0.027" rpy="0 0 0"/>
+            <origin xyz="0 0 0.0425" rpy="0 0 0"/>
         </xacro:inertial_cylinder>
     </link>
@@ -77,5 +77,5 @@
         <parent link="chassis"/>
         <child link="right_wheel"/>
-        <origin xyz="0 -0.1016 0" rpy="${pi/2} 0 0"/>
+        <origin xyz="0 -0.1016 0.00425" rpy="${pi/2} 0 0"/>
         <axis xyz="0 0 -1"/>
     </joint>
@@ -93,5 +93,5 @@
         </collision>
         <xacro:inertial_cylinder mass="0.1" length="0.0254" radius="0.034">
-            <origin xyz="0 0 0.027" rpy="0 0 0"/>
+            <origin xyz="0 0 0.00425" rpy="0 0 0"/>
         </xacro:inertial_cylinder>
     </link>
@@ -103,10 +103,10 @@
         <parent link="chassis"/>
         <child link="caster_wheel"/>
-        <origin xyz="0.24 0 0"/>
+        <origin xyz="0.05 0 -0.023"/>
     </joint>
     <link name="caster_wheel">
         <visual>
             <geometry>
-                <sphere radius="0.05"/>
+                <sphere radius="0.007"/>
             </geometry>
             <material name="black"/>
@@ -114,9 +114,9 @@
         <collision>
             <geometry>
-                <sphere radius="0.05"/>
+                <sphere radius="0.007"/>
             </geometry>
         </collision>
-        <xacro:inertial_sphere mass="0.1" radius="0.05">
-            <origin xyz="0 0 0" rpy="0 0 0"/>
+        <xacro:inertial_sphere mass="0.01" radius="0.007">
+            <origin xyz="0.05 0 -0.023" rpy="0 0 0"/>
         </xacro:inertial_sphere>
     </link>

Commit message: lidar

File: description/lidar.xacro (robot description, xacro)
@@ -4,5 +4,5 @@
         <parent link="chassis"/>
         <child link="laser_frame"/>
-        <origin xyz="0.03 0 0.065" rpy="-${pi} 0 0"/>
+        <origin xyz="0.03 0 0.065" rpy="${pi} 0 ${pi}"/>
     </joint>
     <link name="laser_frame">
